File: ESP_Edgedevice.kicad_sch (KiCad schematic)
At the start: 1 part, among them J1 Screw_Terminal_01x03

Commit message: done
Other:
- sheet Relay ports: added none; removed GND
Changed lines of the file:
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@@
+	(wire
+		(pts
+			(xy 191.77 129.54) (xy 199.39 129.54)
+		)
+		(stroke
+			(width 0)
+			(type default)
+		)
+	)
 	(wire
 		(pts
@@
 		)
 	)
-	(wire
-		(pts
-			(xy 191.77 132.08) (xy 199.39 132.08)
-		)
-		(stroke
-			(width 0)
-			(type default)
-		)
-	)
-	(wire
-		(pts
-			(xy 191.77 135.89) (xy 199.39 135.89)
-		)
-		(stroke
-			(width 0)
-			(type default)
-		)
-	)
 	(global_label "NO"
 		(shape passive)
@@
 	(global_label "INPUT"
 		(shape passive)
-		(at 191.77 135.89 180)
-		(fields_autoplaced yes)
-		(effects
-			(font
-				(size 1.27 1.27)
-			)
-			(justify right)
-		)
-		(property "Intersheetrefs" "${INTERSHEET_REFS}"
-			(at 184.3927 135.89 0)
-			(effects
-				(font
-					(size 1.27 1.27)
-				)
-				(justify right)
-				(hide yes)
-			)
-		)
-	)
-	(global_label "GND"
-		(shape passive)
-		(at 191.77 132.08 180)
-		(fields_autoplaced yes)
-		(effects
-			(font
-				(size 1.27 1.27)
-			)
-			(justify right)
-		)
-		(property "Intersheetrefs" "${INTERSHEET_REFS}"
-			(at 186.0256 132.08 0)
+		(at 191.77 129.54 180)
+		(fields_autoplaced yes)
+		(effects
+			(font
+				(size 1.27 1.27)
+			)
+			(justify right)
+		)
+		(property "Intersheetrefs" "${INTERSHEET_REFS}"
+			(at 184.3927 129.54 0)
 			(effects
 				(font
@@
 			)
 		)
-		(pin "GND" passive
-			(at 199.39 132.08 180)
-			(effects
-				(font
-					(size 1.27 1.27)
-				)
-				(justify left)
-			)
-		)
 		(pin "INPUT" passive
-			(at 199.39 135.89 180)
-			(effects
-				(font
+			(at 199.39 129.54 180)
+			(effects
+				(font

Commit message: modification
Parts:
- added H1: WIZ850IO, WIZ850IO:WIZ850IO, symbol WIZ850IO:WIZ850IO
- added H2, H3, H4, H5: MountingHole, symbol Mechanical:MountingHole
- added J3: Screw_Terminal_01x02, symbol Connector:Screw_Terminal_01x02
- added J3, J4: Conn_01x04_Socket, symbol Connector:Conn_01x04_Socket
- added PS1: HLK-5M05, Converter_ACDC:Converter_ACDC_Hi-Link_HLK-5Mxx, symbol Converter_ACDC:HLK-5M05
- added R3, R4: 10K, symbol Device:R
- added U2: ESP32_NODEMCU, ESP32_NODEMCU:MODULE_ESP32_NODEMCU, symbol ESP32_NODEMCU:ESP32_NODEMCU
Connections:
- net INPUT: now also U2.J5_11 (G25)
- net VCC: now also J3.1 (Pin_1), PS1.4 (+Vout), U2.J5_1 (5V)
- new net AC sensing: U2.J5_15 (G34)
- new net CS: H1.5 (SCNN), U2.J4_10 (G5)
- new net CTa: J4.3 (Pin_3)
- new net CTb: J4.4 (Pin_4)
- new net GND: H1.1 (GND_1), H1.2 (GND_2), H1.7 (GND_3), J3.4 (Pin_4), PS1.3 (-Vout), U2.J4_1 (GND_1), U2.J4_7 (GND_7), U2.J5_6 (GND_6)
- new net INT: H1.6 (INTN), R3.2, U2.J5_7 (G12)
- new net LIVE: J3.1 (Pin_1), J4.1 (Pin_1), PS1.1 (AC/L)
- new net MISO: H1.12 (MISO), U2.J4_8 (G19)
- new net MOSI: H1.3 (MOSI), U2.J4_2 (G23)
- new net NEUTRAL: J3.2 (Pin_2), J4.2 (Pin_2), PS1.2 (AC/N)
- new net RESET: H1.11 (RSTN), R4.2, U2.J4_13 (G4)
- new net RX: J3.2 (Pin_2), U2.J4_11 (G17)
- new net SCK: H1.4 (SCLK), U2.J4_9 (G18)
- new net TX: J3.3 (Pin_3), U2.J4_12 (G16)
- new net VCC_3.3: H1.8 (3.3V_1), H1.9 (3.3V_2), R3.1, R4.1, U2.J5_19 (3V3)
- no-connect marks 0 -> 23
Other:
- added sheet Voltage Sensing (voltagesensing.kicad_sch)
- note added: "AMC1200 based voltage sensing"
- note added: "Ethernet"
- note added: "Hilink 5v/5W powersupply"
- note added: "Relay part"
- moved on the sheet: J1

Commit message: Schematic Editing Done
Parts:
- renumbered J3 to J1, J1 to J2, R3 to R1, R4 to R2, U2 to U1
Other:
- moved on the sheet: J3, J4

Commit message: Assignment Of Footprint Done
Parts:
- removed J2: Screw_Terminal_01x03, symbol Connector:Screw_Terminal_01x03
- removed J3: Screw_Terminal_01x02, symbol Connector:Screw_Terminal_01x02
- removed J4: Conn_01x04_Socket, symbol Connector:Conn_01x04_Socket
- added J2: HB9500-9.5-3P, HB9500-9.5-3P:CONN-TH_HB9500-9.5-3P, symbol HB9500-9.5-3P:HB9500-9.5-3P
- added J3: Barrier Terminal, SparkFun-Connector:Terminal_Block_9.5mm-2, symbol SparkFun-Connector:Barrier_Terminal_9.5mm-2
- added J4: Screw_Terminal_01x04, TerminalBlock:TerminalBlock_bornier-4_P5.08mm, symbol Connector:Screw_Terminal_01x04
- H2, H3, H4, H5: footprint (none) -> MountingHole:MountingHole_2.1mm
- J1: footprint (none) -> Connector_PinHeader_2.54mm:PinHeader_1x04_P2.54mm_Horizontal
- R1, R2: footprint (none) -> Resistor_THT:R_Axial_DIN0207_L6.3mm_D2.5mm_P10.16mm_Horizontal
Connections:
- net COM: now also J2.2
- net CTa: now also J4.3 (Pin_3)
- net CTb: now also J4.4 (Pin_4)
- net LIVE: now also J3.1 (Pin_1), J4.1 (Pin_1)
- net NC: now also J2.3
- net NEUTRAL: now also J3.2 (Pin_2), J4.2 (Pin_2)
- net NO: now also J2.1

Commit message: Placement Of Component on PCB Done
Parts:
- removed H4: MountingHole, MountingHole:MountingHole_2.1mm, symbol Mechanical:MountingHole
- removed J1: Conn_01x04_Socket, Connector_PinHeader_2.54mm:PinHeader_1x04_P2.54mm_Horizontal, symbol Connector:Conn_01x04_Socket
- removed J2: HB9500-9.5-3P, HB9500-9.5-3P:CONN-TH_HB9500-9.5-3P, symbol HB9500-9.5-3P:HB9500-9.5-3P
- removed J4: Screw_Terminal_01x04, TerminalBlock:TerminalBlock_bornier-4_P5.08mm, symbol Connector:Screw_Terminal_01x04
- added J1: HB9500-9.5-3P, HB9500-9.5-3P:CONN-TH_HB9500-9.5-3P, symbol HB9500-9.5-3P:HB9500-9.5-3P
- added U2: PZEM-004T, PZEM-004T:PZEM-004T V3, symbol PZEM-004T:PZEM-004T
- renumbered J3 to J2
Connections:
- net COM: now also J1.2
- net GND: now also U2.1 (GND)
- net LIVE: now also J2.2 (Pin_2), U2.8 (AC-L); no longer J2.1 (Pin_1)
- net NC: now also J1.3
- net NEUTRAL: now also J2.1 (Pin_1), U2.7 (AC-N); no longer J2.2 (Pin_2)
- net NO: now also J1.1
- net RX: now also U2.3 (RX)
- net TX: now also U2.2 (TX)
- net VCC: now also U2.4 (VCC)
- no-connect marks 23 -> 25

Commit message: PCB Routing Completed
Changed lines of the file:
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@@
-	(symbol
-		(lib_id "Mechanical:MountingHole")
-		(at 157.48 175.26 0)
-		(unit 1)
-		(exclude_from_sim no)
-		(in_bom no)
-		(on_board yes)
-		(dnp no)
-		(fields_autoplaced yes)
-		(property "Reference" "H3"
-			(at 160.02 173.9899 0)
-			(effects
-				(font
-					(size 1.27 1.27)
-				)
-				(justify left)
-			)
-		)
-		(property "Value" "MountingHole"
-			(at 160.02 176.5299 0)
-			(effects
-				(font
-					(size 1.27 1.27)
-				)
-				(justify left)
-			)
-		)
-		(property "Footprint" "MountingHole:MountingHole_2.1mm"
-			(at 157.48 175.26 0)
-			(effects
-				(font
-					(size 1.27 1.27)
-				)
-				(hide yes)
-			)
-		)
-		(property "Datasheet" "~"
-			(at 157.48 175.26 0)
-			(effects
-				(font
-					(size 1.27 1.27)
-				)
-				(hide yes)
-			)
-		)
-		(property "Description" "Mounting Hole without connection"
-			(at 157.48 175.26 0)
-			(effects
-				(font
-					(size 1.27 1.27)
-				)
-				(hide yes)
-			)
-		)
-		(instances
-			(project "ESP_Edgedevice"
-				(path "/8fa9f2a2-260d-4024-b3c1-a0bc52ef0867"
-					(reference "H3")
-					(unit 1)
-				)
-			)
-		)
-	)
 	(symbol
 		(lib_id "Mechanical:MountingHole")
@@
 					(unit 1)
 				)
+			)
+		)
+	)
+	(symbol
+		(lib_id "Mechanical:MountingHole")
+		(at 157.48 176.53 0)
+		(unit 1)
+		(exclude_from_sim no)
+		(in_bom no)
+		(on_board yes)
+		(dnp no)
+		(fields_autoplaced yes)
+		(property "Reference" "H3"
+			(at 160.02 175.2599 0)
+			(effects
+				(font
+					(size 1.27 1.27)
+				)
+				(justify left)
+			)
+		)
+		(property "Value" "MountingHole"
+			(at 160.02 177.7999 0)
+			(effects
+				(font
+					(size 1.27 1.27)
+				)
+				(justify left)
+			)
+		)
+		(property "Footprint" "MountingHole:MountingHole_2.1mm"
+			(at 157.48 176.53 0)
+			(effects
+				(font
+					(size 1.27 1.27)
+				)
+				(hide yes)
+			)
+		)
+		(property "Datasheet" "~"
+			(at 157.48 176.53 0)
+			(effects
+				(font
+					(size 1.27 1.27)
+				)
+				(hide yes)
+			)
+		)
+		(property "Description" "Mounting Hole without connection"
+			(at 157.48 176.53 0)
+			(effects
+				(font
+					(size 1.27 1.27)
+				)
+				(hide yes)
+			)
+		)
+		(instances
+			(project "ESP_Edgedevice"
+				(path "/8fa9f2a2-260d-4024-b3c1-a0bc52ef0867"
+					(reference "H3")
+					(unit 1)
+				)
