File: ESP_Edgedevice.kicad_pcb (KiCad board)
At the start: 2 copper layers, 117 x 93 mm, 38 parts, among them J1 HB9500-9.5-3P, J2 Barrier Terminal, J3 Conn_01x02_Pin, K1 SLA-05VDC-SL-C, Q1 S8050, U1 ESP32_NODEMCU, U2 PZEM-004T, U3 PC817X3NSZ1B, U4 AMS1117-5.0, U5 AMC1200SDUBR

Commit message: PCB Routing Completed
Parts:
- moved R3 62.4 mm to (104.3, 84.0), turned to 180 degrees
- moved J3 61.4 mm to (117.2, 82.5), turned to 90 degrees
- moved U3 50.6 mm to (110.5, 81.2), turned to 180 degrees
- moved R4 50.3 mm to (104.3, 81.0), turned to 180 degrees
- moved J2 30.8 mm to (131.7, 36.2)
- moved PS1 29.6 mm to (137.8, 46.0)
- moved D2 26.9 mm to (101.2, 76.5)
- moved Q1 26.5 mm to (94.7, 77.4)
- moved K1 26.1 mm to (101.8, 67.8)
- moved J1 22.8 mm to (110.0, 36.0)
- moved D1 22.4 mm to (120.0, 77.5), turned to 180 degrees
- moved R1 19.9 mm to (149.4, 106.0), turned to 0 degrees
- moved H5 11.8 mm to (162.8, 109.0)
- moved R8 10.2 mm to (199.1, 29.8), turned to 180 degrees
- moved R11 8.50 mm to (190.0, 33.5)
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Connections:
- net Net-(D2-A) renamed /Relay/Relay
Routing:
- net NEUTRAL: track 0.00 -> 218.9 mm
- net /INT: track 0.00 -> 146.7 mm, vias 0 -> 2
- net VCC: track 0.00 -> 124.0 mm
- net VCC_3.3: track 0.00 -> 118.9 mm
- net /RESET: track 0.00 -> 91.5 mm, vias 0 -> 1
- net /CS: track 0.00 -> 90.4 mm
- net /SCK: track 0.00 -> 87.2 mm, vias 0 -> 1
- net LIVE: track 0.00 -> 82.8 mm
- net /MOSI: track 0.00 -> 68.0 mm, vias 0 -> 1
- net /MISO: track 0.00 -> 68.0 mm
- net AC sensing: track 0.00 -> 60.9 mm
- net /TX: track 0.00 -> 59.0 mm
- net /Voltage Sensing/VDD1: track 0.00 -> 53.4 mm
- net /RX: track 0.00 -> 52.9 mm
- net Net-(U5-VINN): track 0.00 -> 52.8 mm
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- added copper zone on B.Cu, net GND
Other:
- outline, holes or cut-outs redrawn
- board text added: "3.3"
- board text added: "5V"
- board text added: "COM"
- board text added: "CS"
- board text added: "GND"
- board text added: "INT"
- board text added: "LIVE"
- board text added: "MISO"
- board text added: "MOSI"
- board text added: "NC"
- board text added: "NEUTRAL"
- board text added: "NO"
- board text added: "RESET"
- board text added: "RX"
- board text added: "SCK"
- board text added: "TX"
- board text added: "VCC"

Commit message: FINAL COMMIT
Parts:
- added G***: LOGO, Libraries:logo, F.Cu at (102.9, 100.0)
- C2: footprint Capacitor_THT:CP_Radial_D5.0mm_P2.50mm -> Capacitor_THT:CP_Radial_D10.0mm_P5.00mm
- moved D4 13.1 mm to (193.2, 45.5), turned to 0 degrees
- moved C2 11.6 mm to (199.6, 38.0)
- moved H3 10.0 mm to (194.0, 49.5)
- moved R6 7.05 mm to (201.2, 30.8), turned to 180 degrees
- moved R8 3.31 mm to (201.2, 27.2)
- moved R7 2.93 mm to (201.3, 24.0)
- moved R5 1.95 mm to (205.2, 24.1)
- moved D3 1.82 mm to (204.8, 42.5), turned to 180 degrees
- moved H5 0.50 mm to (163.2, 109.0)
- renumbered PS1 to HLK-5M05, J3 to Jd_VCC
Routing:
- net NEUTRAL: track 218.9 -> 186.1 mm
- net Net-(D4-K): track 47.3 -> 19.1 mm
- net Net-(D3-K): track 52.6 -> 76.3 mm
- net Net-(C1-Pad1): track 22.3 -> 28.0 mm
- net Net-(R11-Pad1): track 4.17 -> 7.38 mm
- net LIVE: track 82.8 -> 80.9 mm

Commit message: Fix: Corrected Schematic and Updated PCB Layout
Parts:
- added R13: 1K, Resistor_THT:R_Axial_DIN0207_L6.3mm_D2.5mm_P10.16mm_Horizontal, F.Cu at (149.4, 109.0)
- moved J3 5.76 mm to (117.0, 76.8)
- moved D1 4.01 mm to (119.8, 81.5)
- moved PS1 0.30 mm to (137.8, 45.6)
- renumbered Jd_VCC to J3, HLK-5M05 to PS1
Connections:
- D1 pad 1: GND -> Net-(D1-K)
- D1 pad 2: Net-(D1-A) -> INPUT
- U3 pad 2: Net-(D1-A) -> GND
Routing:
- net Net-(D1-K): track 0.00 -> 95.0 mm, vias 0 -> 4
- net INPUT: track 19.5 -> 24.0 mm
- net Net-(D1-A): track 4.20 -> 0.00 mm
- net /MOSI: track 68.0 -> 69.4 mm
- net /Relay/Jd_VCC: track 28.5 -> 29.8 mm
