File: relay.kicad_sch (KiCad schematic)
At the start: 8 parts, among them J2 Conn_01x02_Pin, K2 SLA-05VDC-SL-C, Q1 S8050, U1 PC817X3NSZ1B

Commit message: done
Changed lines of the file:
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@@
-	)
-	(junction
-		(at 161.29 73.66)
-		(diameter 0)
-		(color 0 0 0 0)
-	)
-	(junction
-		(at 121.92 118.11)
-		(diameter 0)
-		(color 0 0 0 0)
-	)
-	(junction
-		(at 121.92 73.66)
-		(diameter 0)
-		(color 0 0 0 0)
 	)
 	(junction
@@
 	(wire
 		(pts
-			(xy 121.92 114.3) (xy 121.92 118.11)
-		)
-		(stroke
-			(width 0)
-			(type default)
-		)
-	)
-	(wire
-		(pts
 			(xy 140.97 113.03) (xy 140.97 106.68)
 		)
@@
 	(wire
 		(pts
-			(xy 153.67 73.66) (xy 161.29 73.66)
-		)
-		(stroke
-			(width 0)
-			(type default)
-		)
-	)
-	(wire
-		(pts
-			(xy 161.29 67.31) (xy 161.29 73.66)
-		)
-		(stroke
-			(width 0)
-			(type default)
-		)
-	)
-	(wire
-		(pts
-			(xy 161.29 73.66) (xy 166.37 73.66)
+			(xy 153.67 73.66) (xy 166.37 73.66)
 		)
 		(stroke
@@
 	(wire
 		(pts
-			(xy 121.92 118.11) (xy 121.92 123.19)
-		)
-		(stroke
-			(width 0)
-			(type default)
-		)
-	)
-	(wire
-		(pts
-			(xy 116.84 99.06) (xy 116.84 118.11)
+			(xy 121.92 114.3) (xy 121.92 123.19)
 		)
 		(stroke
@@
 	(wire
 		(pts
-			(xy 116.84 73.66) (xy 121.92 73.66)
+			(xy 116.84 73.66) (xy 140.97 73.66)
 		)
 		(stroke
@@
 	(wire
 		(pts
-			(xy 121.92 73.66) (xy 140.97 73.66)
-		)
-		(stroke
-			(width 0)
-			(type default)
-		)
-	)
-	(wire
-		(pts
 			(xy 107.95 95.25) (xy 121.92 95.25)
 		)
@@
 	(wire
 		(pts
-			(xy 107.95 99.06) (xy 116.84 99.06)
-		)
-		(stroke
-			(width 0)
-			(type default)
-		)
-	)
-	(wire
-		(pts
-			(xy 121.92 67.31) (xy 121.92 73.66)
-		)
-		(stroke
-			(width 0)
-			(type default)
-		)
-	)
-	(wire
-		(pts
 			(xy 166.37 101.6) (xy 170.18 101.6)
 		)
@@
 	(wire
 		(pts
-			(xy 116.84 118.11) (xy 121.92 118.11)
-		)
-		(stroke
-			(width 0)
-			(type default)
-		)
-	)
-	(wire
-		(pts
 			(xy 161.29 93.98) (xy 166.37 93.98)
 		)
@@
 			(width 0)
 			(type default)
-		)
-	)
-	(label "VCC"
-		(at 116.84 73.66 180)
-		(effects
-			(font
-				(size 1.27 1.27)
-			)
-			(justify right bottom)
 		)
 	)
@@
 		(shape passive)
 		(at 107.95 95.25 180)
-		(effects
-			(font
-				(size 1.27 1.27)
-			)
-			(justify right)
-		)
-	)
-	(hierarchical_label "GND"
-		(shape passive)
-		(at 107.95 99.06 180)
 		(effects
 			(font
@@
 	)
 	(symbol
-		(lib_id "power:PWR_FLAG")
-		(at 161.29 67.31 0)
-		(unit 1)
-		(exclude_from_sim no)
-		(in_bom yes)
-		(on_board yes)
-		(dnp no)
-		(fields_autoplaced yes)
-		(property "Reference" "#FLG02"
-			(at 161.29 65.405 0)
-			(effects
-				(font
-					(size 1.27 1.27)
-				)
-				(hide yes)
-			)
-		)
-		(property "Value" "PWR_FLAG"
-			(at 161.29 62.23 0)
-			(effects
-				(font
-					(size 1.27 1.27)
-				)
-			)
-		)
-		(property "Footprint" ""
-			(at 161.29 67.31 0)
-			(effects
-				(font
-					(size 1.27 1.27)
-				)
-				(hide yes)
-			)
-		)
-		(property "Datasheet" "~"
-			(at 161.29 67.31 0)
-			(effects
-				(font
-					(size 1.27 1.27)
-				)
-				(hide yes)
-			)
-		)
-		(property "Description" "Special symbol for telling ERC where power comes from"
-			(at 161.29 67.31 0)
-			(effects
-				(font
-					(size 1.27 1.27)
-				)
-				(hide yes)
-			)
-		)
-		(pin "1"
-		)
-		(instances
-			(project "ESP_Edgedevice"
-				(path "/8fa9f2a2-260d-4024-b3c1-a0bc52ef0867/c380d0b5-0235-468c-a489-737f32e01687"
-					(reference "#FLG02")
-					(unit 1)
-				)
-			)
-		)
-	)
-	(symbol
 		(lib_id "SLA-05VDC-SL-C:SLA-05VDC-SL-C")
 		(at 170.18 93.98 0)
@@
 					(unit 1)
 				)
-			)
-		)
-	)
-	(symbol
-		(lib_id "power:PWR_FLAG")
-		(at 121.92 67.31 0)
-		(unit 1)
-		(exclude_from_sim no)
-		(in_bom yes)
-		(on_board yes)
-		(dnp no)
-		(fields_autoplaced yes)
-		(property "Reference" "#FLG01"
-			(at 121.92 65.405 0)
-			(effects
-				(font
-					(size 1.27 1.27)
-				)
-				(hide yes)
-			)
-		)
-		(property "Value" "PWR_FLAG"
-			(at 121.92 62.23 0)
-			(effects
-				(font
-					(size 1.27 1.27)
-				)
-			)
-		)
-		(property "Footprint" ""
-			(at 121.92 67.31 0)
-			(effects
-				(font
-					(size 1.27 1.27)
-				)
-				(hide yes)
-			)
-		)
-		(property "Datasheet" "~"
-			(at 121.92 67.31 0)
-			(effects
-				(font
-					(size 1.27 1.27)
-				)
-				(hide yes)
-			)
-		)
-		(property "Description" "Special symbol for telling ERC where power comes from"
-			(at 121.92 67.31 0)
-			(effects
-				(font
-					(size 1.27 1.27)
-				)
-				(hide yes)
-			)
-		)
-		(pin "1"
-		)
-		(instances
-			(project ""
-				(path "/8fa9f2a2-260d-4024-b3c1-a0bc52ef0867/c380d0b5-0235-468c-a489-737f32e01687"
-					(reference "#FLG01")
-					(unit 1)
-				)

Commit message: modification
Parts:
- renumbered D1 to D, D2 to D, J2 to J, K2 to K, Q1 to Q, R2 to R, U1 to U
Changed lines of the file:
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@@
 		(dnp no)
 		(fields_autoplaced yes)
-		(property "Reference" "D1"
+		(property "Reference" "D"
 			(at 125.73 110.8074 90)
 			(effects
@@
 		(pin "2"
 		)
-		(instances
-			(project ""
-				(path "/8fa9f2a2-260d-4024-b3c1-a0bc52ef0867/c380d0b5-0235-468c-a489-737f32e01687"
-					(reference "D1")
-					(unit 1)
-				)
-			)
-		)
+		(instances)
 	)
 	(symbol
@@
 		(dnp no)
 		(fields_autoplaced yes)
-		(property "Reference" "K2"
+		(property "Reference" "K"
 			(at 182.88 86.36 0)
 			(effects
@@
 		(pin "3"
 		)
-		(instances
-			(project ""
-				(path "/8fa9f2a2-260d-4024-b3c1-a0bc52ef0867/c380d0b5-0235-468c-a489-737f32e01687"
-					(reference "K2")
-					(unit 1)
-				)
-			)
-		)
+		(instances)
 	)
 	(symbol
@@
 		(dnp no)
 		(fields_autoplaced yes)
-		(property "Reference" "R2"
+		(property "Reference" "R"
 			(at 125.73 88.9 90)
 			(effects
@@
 		(pin "2"
 		)
-		(instances
-			(project ""
-				(path "/8fa9f2a2-260d-4024-b3c1-a0bc52ef0867/c380d0b5-0235-468c-a489-737f32e01687"
-					(reference "R2")
-					(unit 1)
-				)
-			)
-		)
+		(instances)
 	)
 	(symbol
@@
 		(dnp no)
 		(fields_autoplaced yes)
-		(property "Reference" "#PWR01"
+		(property "Reference" "#PWR"
 			(at 161.29 130.81 0)
 			(effects
@@
 		(pin "1"
 		)
-		(instances
-			(project ""
-				(path "/8fa9f2a2-260d-4024-b3c1-a0bc52ef0867/c380d0b5-0235-468c-a489-737f32e01687"
-					(reference "#PWR01")
-					(unit 1)
-				)
-			)
-		)
+		(instances)
 	)
 	(symbol
@@
 		(on_board yes)
 		(dnp no)
-		(property "Reference" "J2"
+		(property "Reference" "J"
 			(at 135.89 71.12 90)
 			(effects
@@
 		(pin "1"
 		)
-		(instances
-			(project ""
-				(path "/8fa9f2a2-260d-4024-b3c1-a0bc52ef0867/c380d0b5-0235-468c-a489-737f32e01687"
-					(reference "J2")
-					(unit 1)
-				)
-			)
-		)
+		(instances)
 	)
 	(symbol
@@
 		(dnp no)
 		(fields_autoplaced yes)
-		(property "Reference" "Q1"
+		(property "Reference" "Q"
 			(at 163.83 111.7599 0)
 			(effects
@@
 		(pin "1"
 		)
-		(instances
-			(project ""
-				(path "/8fa9f2a2-260d-4024-b3c1-a0bc52ef0867/c380d0b5-0235-468c-a489-737f32e01687"
-					(reference "Q1")
-					(unit 1)
-				)
-			)
-		)
+		(instances)
 	)
 	(symbol
@@
 		(dnp no)
 		(fields_autoplaced yes)
-		(property "Reference" "U1"
+		(property "Reference" "U"
 			(at 140.97 87.63 0)
 			(effects
@@
 		(pin "4"
 		)
-		(instances
-			(project ""
-				(path "/8fa9f2a2-260d-4024-b3c1-a0bc52ef0867/c380d0b5-0235-468c-a489-737f32e01687"
-					(reference "U1")
-					(unit 1)
-				)
-			)
-		)
+		(instances)
 	)
 	(symbol
@@
 		(on_board yes)
 		(dnp no)
-		(property "Reference" "D2"
+		(property "Reference" "D"
 			(at 160.02 88.9 90)
 			(effects
@@
 		(pin "1"
 		)
-		(instances
-			(project ""
-				(path "/8fa9f2a2-260d-4024-b3c1-a0bc52ef0867/c380d0b5-0235-468c-a489-737f32e01687"
-					(reference "D2")
-					(unit 1)
-				)
-			)
-		)
+		(instances)
 	)
 )

Commit message: Schematic Editing Done
Parts:
- removed K: SLA-05VDC-SL-C, K_SLA_C_NFR, symbol SLA-05VDC-SL-C:SLA-05VDC-SL-C
- added K1: SLA-05VDC-SL-C, K_SLA_C_NFR, symbol SLA-05VDC-SL-C:SLA-05VDC-SL-C
- renumbered D to D1, D to D2, J to J5, Q to Q1, R to R3, R1 to R4, U to U2
Connections:
- net COM: now also K1.3, K1.4
- net Jd_VCC: now also K1.1
- net NC: now also K1.6
- net NO: now also K1.5
- net at D2.2 (A), Q1.3 (C): now also K1.2
Changed lines of the file:
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@@
 		(dnp no)
 		(fields_autoplaced yes)
-		(property "Reference" "#PWR02"
+		(property "Reference" "#PWR04"
 			(at 121.92 129.54 0)
 			(effects
@@
 			(project "ESP_Edgedevice"
 				(path "/8fa9f2a2-260d-4024-b3c1-a0bc52ef0867/c380d0b5-0235-468c-a489-737f32e01687"
-					(reference "#PWR02")
+					(reference "#PWR04")
 					(unit 1)
 				)
@@
 		(dnp no)
 		(fields_autoplaced yes)
-		(property "Reference" "D"
+		(property "Reference" "D1"
 			(at 125.73 110.8074 90)
 			(effects
@@
 		(pin "2"
 		)
-		(instances)
+		(instances
+			(project "ESP_Edgedevice"
+				(path "/8fa9f2a2-260d-4024-b3c1-a0bc52ef0867/c380d0b5-0235-468c-a489-737f32e01687"
+					(reference "D1")
+					(unit 1)
+				)
+			)
+		)
 	)
 	(symbol
@@
 		(on_board yes)
 		(dnp no)
-		(property "Reference" "R1"
+		(property "Reference" "R4"
 			(at 148.59 115.57 90)
 			(effects
@@
 			(project "ESP_Edgedevice"
 				(path "/8fa9f2a2-260d-4024-b3c1-a0bc52ef0867/c380d0b5-0235-468c-a489-737f32e01687"
-					(reference "R1")
+					(reference "R4")
 					(unit 1)
 				)
@@
 		(dnp no)
 		(fields_autoplaced yes)
-		(property "Reference" "K"
+		(property "Reference" "K1"
 			(at 182.88 86.36 0)
 			(effects
@@
 			)
 		)
-		(property "Datasheet" "kicad-embed://SLA-05VDC-SL-A.pdf"
+		(property "Datasheet" "SLA-05VDC-SL-C"
 			(at 170.18 93.98 0)
 			(effects
@@
 			)
 		)
+		(pin "5"
+		)
+		(pin "2"
+		)
+		(pin "6"
+		)
 		(pin "4"
 		)
-		(pin "5"
-		)
-		(pin "6"
-		)
-		(pin "2"
-		)
-		(pin "1"
-		)
 		(pin "3"
 		)
-		(instances)
+		(pin "1"
+		)
+		(instances
+			(project ""
+				(path "/8fa9f2a2-260d-4024-b3c1-a0bc52ef0867/c380d0b5-0235-468c-a489-737f32e01687"
+					(reference "K1")
+					(unit 1)
+				)
+			)
+		)
 	)
 	(symbol
@@
 		(dnp no)
 		(fields_autoplaced yes)
-		(property "Reference" "R"
+		(property "Reference" "R3"
 			(at 125.73 88.9 90)
 			(effects
@@
 		(pin "2"
 		)
-		(instances)
+		(instances
+			(project "ESP_Edgedevice"
+				(path "/8fa9f2a2-260d-4024-b3c1-a0bc52ef0867/c380d0b5-0235-468c-a489-737f32e01687"
+					(reference "R3")
+					(unit 1)
+				)
+			)
+		)
 	)
 	(symbol
@@
 		(dnp no)
 		(fields_autoplaced yes)
-		(property "Reference" "#PWR"
+		(property "Reference" "#PWR05"
 			(at 161.29 130.81 0)
 			(effects
@@
 		(pin "1"
 		)
-		(instances)
+		(instances
+			(project "ESP_Edgedevice"
+				(path "/8fa9f2a2-260d-4024-b3c1-a0bc52ef0867/c380d0b5-0235-468c-a489-737f32e01687"
+					(reference "#PWR05")
+					(unit 1)
+				)
+			)
+		)
 	)
 	(symbol
@@
 		(on_board yes)
 		(dnp no)
-		(property "Reference" "J"
+		(property "Reference" "J5"
 			(at 135.89 71.12 90)
 			(effects
@@
 		(pin "1"
 		)
-		(instances)
+		(instances
+			(project "ESP_Edgedevice"
+				(path "/8fa9f2a2-260d-4024-b3c1-a0bc52ef0867/c380d0b5-0235-468c-a489-737f32e01687"
+					(reference "J5")
+					(unit 1)
+				)
+			)
+		)
 	)
 	(symbol
@@
 		(dnp no)
 		(fields_autoplaced yes)
-		(property "Reference" "Q"
+		(property "Reference" "Q1"
 			(at 163.83 111.7599 0)
 			(effects
@@
 		(pin "1"
 		)
-		(instances)
+		(instances
+			(project "ESP_Edgedevice"
+				(path "/8fa9f2a2-260d-4024-b3c1-a0bc52ef0867/c380d0b5-0235-468c-a489-737f32e01687"
+					(reference "Q1")
+					(unit 1)
+				)
+			)
+		)
 	)
 	(symbol
@@
 		(dnp no)
 		(fields_autoplaced yes)
-		(property "Reference" "U"
+		(property "Reference" "U2"
 			(at 140.97 87.63 0)
 			(effects
@@
 		(pin "4"
 		)
-		(instances)
+		(instances
+			(project "ESP_Edgedevice"
+				(path "/8fa9f2a2-260d-4024-b3c1-a0bc52ef0867/c380d0b5-0235-468c-a489-737f32e01687"
+					(reference "U2")
+					(unit 1)
+				)
+			)
+		)
 	)
 	(symbol
@@
 		(on_board yes)
 		(dnp no)
-		(property "Reference" "D"
+		(property "Reference" "D2"
 			(at 160.02 88.9 90)
 			(effects
@@
 		(pin "1"
 		)
-		(instances)
+		(instances
+			(project "ESP_Edgedevice"
+				(path "/8fa9f2a2-260d-4024-b3c1-a0bc52ef0867/c380d0b5-0235-468c-a489-737f32e01687"
+					(reference "D2")
+					(unit 1)
+				)
+			)
+		)
 	)
 )

Commit message: Assignment Of Footprint Done
Parts:
- removed J5: Conn_01x02_Pin, symbol Connector:Conn_01x02_Pin
- D1: footprint (none) -> LED_THT:LED_D3.0mm
- K1: footprint K_SLA_C_NFR -> SLA-05VDC-SL-C:K_SLA_C_NFR
- R3, R4: footprint (none) -> Resistor_THT:R_Axial_DIN0207_L6.3mm_D2.5mm_P10.16mm_Horizontal
Changed lines of the file:
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@@
 			)
 		)
-		(property "Footprint" ""
+		(property "Footprint" "LED_THT:LED_D3.0mm"
 			(at 121.92 110.49 0)
 			(effects
@@
 			)
 		)
-		(property "Footprint" ""
+		(property "Footprint" "Resistor_THT:R_Axial_DIN0207_L6.3mm_D2.5mm_P10.16mm_Horizontal"
 			(at 148.59 114.808 90)
 			(effects
@@
 			)
 		)
-		(property "Footprint" "K_SLA_C_NFR"
+		(property "Footprint" "SLA-05VDC-SL-C:K_SLA_C_NFR"
 			(at 170.18 93.98 0)
 			(effects
@@
 			)
 		)
-		(property "Footprint" ""
+		(property "Footprint" "Resistor_THT:R_Axial_DIN0207_L6.3mm_D2.5mm_P10.16mm_Horizontal"
 			(at 125.73 97.028 90)
 			(effects
@@
 					(unit 1)
 				)
-			)
-		)
-	)
-	(symbol
-		(lib_id "Connector:Conn_01x02_Pin")
-		(at 143.51 68.58 270)
-		(unit 1)
-		(exclude_from_sim no)
-		(in_bom yes)
-		(on_board yes)
-		(dnp no)
-		(property "Reference" "J5"
-			(at 135.89 71.12 90)
-			(effects
-				(font
-					(size 1.27 1.27)
-				)
-				(justify left)
-			)
-		)
-		(property "Value" "Conn_01x02_Pin"
-			(at 134.62 76.2 90)
-			(effects
-				(font
-					(size 1.27 1.27)
-				)
-				(justify left)
-			)
-		)
-		(property "Footprint" ""
-			(at 143.51 68.58 0)
-			(effects
-				(font
-					(size 1.27 1.27)
-				)
-				(hide yes)
-			)
-		)
-		(property "Datasheet" "~"
-			(at 143.51 68.58 0)
-			(effects
-				(font
-					(size 1.27 1.27)
-				)
-				(hide yes)
-			)
-		)
-		(property "Description" "Generic connector, single row, 01x02, script generated"
-			(at 143.51 68.58 0)
-			(effects
-				(font
-					(size 1.27 1.27)
-				)
-				(hide yes)
-			)
-		)
-		(pin "2"
-		)
-		(pin "1"
-		)
-		(instances
-			(project "ESP_Edgedevice"
-				(path "/8fa9f2a2-260d-4024-b3c1-a0bc52ef0867/c380d0b5-0235-468c-a489-737f32e01687"
-					(reference "J5")
-					(unit 1)
-				)

Commit message: Placement Of Component on PCB Done
Parts:
- added J3: Conn_01x02_Pin, Connector_PinHeader_2.54mm:PinHeader_1x02_P2.54mm_Vertical, symbol Connector:Conn_01x02_Pin
- renumbered U2 to U3
Connections:
- net Jd_VCC: now also J3.1 (Pin_1)
- net VCC: now also J3.2 (Pin_2)
Changed lines of the file:
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@@
 		(dnp no)
 		(fields_autoplaced yes)
-		(property "Reference" "U2"
+		(property "Reference" "U3"
 			(at 140.97 87.63 0)
 			(effects
@@
 			(project "ESP_Edgedevice"
 				(path "/8fa9f2a2-260d-4024-b3c1-a0bc52ef0867/c380d0b5-0235-468c-a489-737f32e01687"
-					(reference "U2")
+					(reference "U3")
 					(unit 1)
 				)
@@
 					(unit 1)
 				)
+			)
+		)
+	)
+	(symbol
+		(lib_id "Connector:Conn_01x02_Pin")
+		(at 143.51 68.58 270)
+		(unit 1)
+		(exclude_from_sim no)
+		(in_bom yes)
+		(on_board yes)
+		(dnp no)
+		(fields_autoplaced yes)
+		(property "Reference" "J3"
+			(at 144.78 67.9449 90)
+			(effects
+				(font
+					(size 1.27 1.27)
+				)
+				(justify left)
+			)
+		)
+		(property "Value" "Conn_01x02_Pin"
+			(at 144.78 70.4849 90)
+			(effects
+				(font
+					(size 1.27 1.27)
+				)
+				(justify left)
+			)
+		)
+		(property "Footprint" "Connector_PinHeader_2.54mm:PinHeader_1x02_P2.54mm_Vertical"
+			(at 143.51 68.58 0)
+			(effects
+				(font
+					(size 1.27 1.27)
+				)
+				(hide yes)
+			)
+		)
+		(property "Datasheet" "~"
+			(at 143.51 68.58 0)
+			(effects
+				(font
+					(size 1.27 1.27)
+				)
+				(hide yes)
+			)
+		)
+		(property "Description" "Generic connector, single row, 01x02, script generated"
+			(at 143.51 68.58 0)
+			(effects
+				(font
+					(size 1.27 1.27)
+				)
+				(hide yes)
+			)
+		)
+		(pin "1"
+		)
+		(pin "2"
+		)
+		(instances
+			(project ""
+				(path "/8fa9f2a2-260d-4024-b3c1-a0bc52ef0867/c380d0b5-0235-468c-a489-737f32e01687"
+					(reference "J3")
+					(unit 1)
+				)

Commit message: PCB Routing Completed
Connections:
- net Relay: now reaches D2.2 (A), K1.2, Q1.3 (C)
Changed lines of the file:
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@@
+		)
+	)
+	(label "Relay"
+		(at 163.83 101.6 0)
+		(effects
+			(font
+				(size 1.27 1.27)
+			)
+			(justify left bottom)
 		)
 	)

Commit message: Fix: Corrected Schematic and Updated PCB Layout
Parts:
- added R13: 1K, Resistor_THT:R_Axial_DIN0207_L6.3mm_D2.5mm_P10.16mm_Horizontal, symbol Device:R
Connections:
- net GND: now also U3.2, R13.2; no longer D1.1 (K)
- net INPUT: now also D1.2 (A)
- new net: D1.1 (K), R13.1
Other:
- moved on the sheet: D1
Changed lines of the file:
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@@
+	)
+	(junction
+		(at 115.57 95.25)
+		(diameter 0)
+		(color 0 0 0 0)
 	)
 	(junction
@@
 	)
 	(junction
+		(at 121.92 115.57)
+		(diameter 0)
+		(color 0 0 0 0)
+	)
+	(junction
 		(at 166.37 93.98)
 		(diameter 0)
@@
 	(wire
 		(pts
+			(xy 115.57 105.41) (xy 115.57 102.87)
+		)
+		(stroke
+			(width 0)
+			(type default)
+		)
+	)
+	(wire
+		(pts
 			(xy 166.37 93.98) (xy 170.18 93.98)
 		)
@@
 	(wire
 		(pts
+			(xy 115.57 115.57) (xy 121.92 115.57)
+		)
+		(stroke
+			(width 0)
+			(type default)
+		)
+	)
+	(wire
+		(pts
+			(xy 121.92 100.33) (xy 121.92 115.57)
+		)
+		(stroke
+			(width 0)
+			(type default)
+		)
+	)
+	(wire
+		(pts
 			(xy 140.97 113.03) (xy 144.78 113.03)
 		)
@@
 	(wire
 		(pts
-			(xy 121.92 106.68) (xy 121.92 100.33)
-		)
-		(stroke
-			(width 0)
-			(type default)
-		)
-	)
-	(wire
-		(pts
 			(xy 195.58 96.52) (xy 196.85 96.52)
 		)
@@
 	(wire
 		(pts
+			(xy 121.92 115.57) (xy 121.92 123.19)
+		)
+		(stroke
+			(width 0)
+			(type default)
+		)
+	)
+	(wire
+		(pts
 			(xy 140.97 113.03) (xy 140.97 106.68)
 		)
@@
 	(wire
 		(pts
-			(xy 121.92 114.3) (xy 121.92 123.19)
+			(xy 116.84 73.66) (xy 140.97 73.66)
 		)
 		(stroke
@@
 	(wire
 		(pts
-			(xy 116.84 73.66) (xy 140.97 73.66)
+			(xy 115.57 113.03) (xy 115.57 115.57)
 		)
 		(stroke
@@
 	(wire
 		(pts
-			(xy 107.95 95.25) (xy 121.92 95.25)
+			(xy 107.95 95.25) (xy 115.57 95.25)
 		)
 		(stroke
@@
 		(pts
 			(xy 151.13 95.25) (xy 153.67 95.25)
+		)
+		(stroke
+			(width 0)
+			(type default)
+		)
+	)
+	(wire
+		(pts
+			(xy 115.57 95.25) (xy 121.92 95.25)
 		)
 		(stroke
@@
 	(symbol
 		(lib_id "Device:LED")
-		(at 121.92 110.49 90)
+		(at 115.57 99.06 90)
 		(unit 1)
 		(exclude_from_sim no)
@@
 		(fields_autoplaced yes)
 		(property "Reference" "D1"
-			(at 125.73 110.8074 90)
+			(at 119.38 99.3774 90)
 			(effects
 				(font
@@
 		)
 		(property "Value" "LED"
-			(at 125.73 113.3474 90)
+			(at 119.38 101.9174 90)
 			(effects
 				(font
@@
 		)
 		(property "Footprint" "LED_THT:LED_D3.0mm"
-			(at 121.92 110.49 0)
+			(at 115.57 99.06 0)
 			(effects
 				(font
@@
 		)
 		(property "Datasheet" "~"
-			(at 121.92 110.49 0)
+			(at 115.57 99.06 0)
 			(effects
 				(font
@@
 		)
 		(property "Description" "Light emitting diode"
-			(at 121.92 110.49 0)
+			(at 115.57 99.06 0)
 			(effects
 				(font
@@
 		)
 		(property "Sim.Pins" "1=K 2=A"
-			(at 121.92 110.49 0)
+			(at 115.57 99.06 0)
 			(effects
 				(font
@@
 					(unit 1)
 				)
+			)
+		)
+	)
+	(symbol
+		(lib_id "Device:R")
+		(at 115.57 109.22 0)
+		(unit 1)
+		(exclude_from_sim no)
+		(in_bom yes)
+		(on_board yes)
+		(dnp no)
+		(property "Reference" "R13"
+			(at 113.03 109.22 90)
+			(effects
+				(font
+					(size 1.27 1.27)
+				)
+			)
+		)
+		(property "Value" "1K"
+			(at 118.11 109.22 90)
+			(effects
+				(font
+					(size 1.27 1.27)
+				)
+			)
+		)
+		(property "Footprint" "Resistor_THT:R_Axial_DIN0207_L6.3mm_D2.5mm_P10.16mm_Horizontal"
+			(at 113.792 109.22 90)
+			(effects
+				(font
+					(size 1.27 1.27)
+				)
+				(hide yes)
+			)
+		)
+		(property "Datasheet" "~"
+			(at 115.57 109.22 0)
+			(effects
+				(font
+					(size 1.27 1.27)
+				)
+				(hide yes)
+			)
+		)
+		(property "Description" "Resistor"
+			(at 115.57 109.22 0)
+			(effects
+				(font
+					(size 1.27 1.27)
+				)
+				(hide yes)
+			)
+		)
+		(pin "1"
+		)
+		(pin "2"
+		)
+		(instances
+			(project "ESP_Edgedevice"
+				(path "/8fa9f2a2-260d-4024-b3c1-a0bc52ef0867/c380d0b5-0235-468c-a489-737f32e01687"
+					(reference "R13")
+					(unit 1)
+				)
